File: electrical/pcb/control_board/Motor_Board.sch (KiCad schematic (older format))
At the start: 89 parts, among them J1 ED2627-ND, J11 S7038-ND_regulator_D24V22F12, J12 PPTC102LFBN-RC, J13 XT60-F, J14 ED2989-ND-USB, J15 XT60-F, J16 XT60-F, J17 Molex_172675-0613, J18 Molex_172675-0613, J19 Molex_172675-0613, J2 ED2627-ND, J20 Molex_172675-0613, J21 Molex_172675-0613, J22 Molex_172675-0613, J28 XT60-F, J29 XT60-F, J3 ED2627-ND, J30 XT60-F, J53 PEC08SAAN, J69 PEC04SAAN_5v_regulator_2, M1 Mounting_Holes, T1 test_point, T2 test_point, T3 test_point, T5 test_point, T6 test_point, y1 rover_silkscreen

Commit message: Editing simple footprint stuff
Parts:
- removed J11: S7038-ND_regulator_D24V22F12, JPL Robotics:S7038-ND_withkeepout, symbol JPL_Robotics_Lib:S7038-ND_regulator_D24V22F12
- removed J69: PEC04SAAN_5v_regulator_2, symbol JPL_Robotics_Lib:PEC04SAAN_5v_regulator_2
- added U?: D24V22Fx, symbol JPL_Robotics_Lib:D24V22Fx
Connections:
- net labels added: EN_12V
- wire segments 420 -> 424
- no-connect marks 56 -> 54
Other:
- moved on the sheet: T5, T6, U?
